File: prelude.sch (KiCad schematic (older format))
At the start: 36 parts, among them J1 CONN_01X50, J2 USB_C, J3 Conn_01x04, J4 Conn_01x08, SW1 SW_Push, U1 LM3671MF-3.3, U2 STM32F411RETx, U3 AP5724, Y1 16MHz

Commit message: Replaces Inductors (L1 and L2) with HandSoldering versions
Parts:
- L1: footprint Inductor_SMD:L_Taiyo-Yuden_NR-24xx -> Inductor_SMD:L_Taiyo-Yuden_NR-24xx_HandSoldering
- L2: footprint Inductor_SMD:L_Taiyo-Yuden_NR-30xx -> Inductor_SMD:L_Taiyo-Yuden_NR-30xx_HandSoldering
Changed lines of the file:
@@
 F 0 "L2" V 7850 750 50  0000 C CNN
 F 1 "22uH" V 7975 750 50  0000 C CNN
-F 2 "Inductor_SMD:L_Taiyo-Yuden_NR-30xx" H 7900 750 50  0001 C CNN
+F 2 "Inductor_SMD:L_Taiyo-Yuden_NR-30xx_HandSoldering" H 7900 750 50  0001 C CNN
 F 3 "" H 7900 750 50  0001 C CNN
 	1    7900 750
@@
 F 0 "L1" V 5550 1000 50  0000 C CNN
 F 1 "2.2uH" V 5675 1000 50  0000 C CNN
-F 2 "Inductor_SMD:L_Taiyo-Yuden_NR-24xx" H 5600 1000 50  0001 C CNN
+F 2 "Inductor_SMD:L_Taiyo-Yuden_NR-24xx_HandSoldering" H 5600 1000 50  0001 C CNN
 F 3 "" H 5600 1000 50  0001 C CNN
 	1    5600 1000
